File: pcb/23XXAdapter_v1.1.sch (EAGLE design)
At the start: 24 parts, among them IC1 EPROM, IC2 74LS138N

Commit message: PCB cleanup and additional images
Parts:
- added R1', R2', R3', R4', R5': (no value), resistor:R-US_R0805
Connections:
- net A11: now also R1'.1, R1.1; no longer R5.1
- net A12: now also R2'.1, R2.1; no longer R1.1
- net A13: now also R3'.1, R3.1; no longer R2.1
- net A14: now also R4'.1, R4.1; no longer R3.1
- net A15: now also R5'.1, R5.1; no longer R4.1
- net VCC: now also R1'.2, R2'.2, R3'.2, R4'.2, R5'.2
Other:
- moved on the sheet: HDR1, IC1, R1, R2, R3, R4, R5
